File: 1_Small_ST-Link/STl-Link-V14.sch (EAGLE design)
At the start: 17 parts

Commit message: V3 Lot of Changes
eagle-files fallback
other programmer
separate pins
optimized layout
Parts:
- removed R5: 560, rcl:R-EU_0204/7
- removed SV2: (no value), con-lsta:FE07-2W
- removed SV3: (no value), con-lstb:MAR05-1
- removed TP5: TPB1,27, testpad:TPB1,27
- added 5V, 5VIN, G, G1, G2, G3, G4, G5, G6, GND, IR+, IR-IN, IR-SEND+, IR-SEND-, LED, PC+, PC-, PWR+, PWR-: (no value), wirepad:SMD2
- added C3: 4,7uF, rcl:C-EUC1206K
- added D1: (no value), diode:DIODE-SOD123
- added PWR, SEND: (no value), led:LEDCHIPLED_1206
- added R9: 220, rcl:R-EU_R0805W
- added SV4: (no value), con-lsta:FE05-1
- added T1: BC847, transistor:BC847
- added X1: 1501_03, con-lumberg:1501_03
- R1, R4: value 100 -> 220
- R2, R3: value 560 -> 100
- R6, R8: value 560 -> 220
- R7: value 560 -> 10; device rcl:R-EU_0204/7 -> rcl:R-EU_R0805W
- renumbered LED1 to TOG
Connections:
- removed net FREE: SV3.1
- removed net IR-SEND: R7.2, R8.2, SV2.14
- removed net N$2: OK2.A, R1.2, R4.2
- removed net N$4: OK2.EMIT, SV2.1, SV2.2
- removed net OK2: OK2.COL, SV2.3, SV2.4
- removed net TCK: SV3.3
- removed net TMS: SV3.5
- new net 5VIN: 5VIN.P, D1.A
- new net IR+: C1.+, C2.1, IR+.P, R2.1, R3.1, X1.3
- new net IR-SEND+: IR-SEND+.P, R7.2
- new net IR-SEND-: IR-SEND-.P, SEND.C, T1.C
- new net N$3: R8.1, T1.B
- new net OK: OK2.A, PWR.A, R1.2, R4.2
- new net PWR+: OK2.COL, PC+.P, PWR+.P
- new net PWR-: OK2.EMIT, PC-.P, PWR-.P
- net 3V3: now also C3.1, R7.1, R9.1, SV4.2; no longer SV2.13, SV2.9, SV3.2
- net 5V: now also 5V.P, D1.C, SV4.1
- net CLK-TOGGLE-LED: now also SV4.3; no longer R5.2
- net DIO-EINSCH: now also SV4.5
- net GND: now also C3.2, G.P, G1.P, G2.P, G3.P, G4.P, G5.P, G6.P, GND.P, PWR.C, SV4.4, T1.E, X1.1; no longer SV2.10, SV2.12, SV2.7, SV3.4
- net LED: now also LED.P; no longer R5.1, SV2.11
- net N$1: now also R9.2, SEND.A; no longer C1.+, C2.1, R2.1, R3.1
- net NRST-IR-SEND: now also R8.2; no longer R7.1, R8.1
- net SWIM-IR-IN: now also IR-IN.P, X1.2; no longer SV2.5, TP5.TP
Other:
- note removed: "+"
- moved on the sheet: R7, R8
