File: 4-SWD-Interface/SWD-IR-V01-003.brd (EAGLE design)
At the start: 11 x 11 mm, 14 parts

Commit message: V003
Parts:
- moved C2 0.92 mm to (13.0, 8.26), turned to 90 degrees
Routing:
- net GND: track 14.5 -> 11.2 mm, vias 1 -> 0
- net SWIM-IR-IN: track 9.43 -> 11.8 mm, vias 0 -> 2
- net CLK: track 7.29 -> 5.39 mm
- net PWR+: track 18.7 -> 19.6 mm
- net IR+: track 13.4 -> 14.2 mm

Commit message: beschriftung
Connections:
- net SWIM-IR-IN renamed IO
Changed lines of the file:
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@@
 <text x="16.0015" y="12.223" size="0.508" layer="25" font="vector">V0.1</text>
 <text x="8.382" y="11.365" size="0.4064" layer="25" font="vector">GND</text>
-<text x="9.398" y="9.209" size="0.4064" layer="25" font="vector" rot="R180">DIO</text>
-<text x="8.382" y="6.285" size="0.4064" layer="25" font="vector">CLK</text>
+<text x="9.398" y="9.209" size="0.4064" layer="25" font="vector" rot="R180">CLK</text>
+<text x="8.382" y="6.285" size="0.4064" layer="25" font="vector">IO</text>
 <text x="9.398" y="11.43" size="0.4064" layer="26" rot="MR0">GND</text>
 <text x="9.398" y="3.81" size="0.4064" layer="26" rot="MR0">VCC</text>
@@
 <wire x1="11.43" y1="9.9425" x2="10.625190625" y2="9.9425" width="0.3048" layer="16"/>
 </signal>
-<signal name="SWIM-IR-IN">
+<signal name="IO">
 <contactref element="IR-IN" pad="1"/>
 <contactref element="SV1" pad="2"/>
